File: 2Key/2Key.kicad_sch (KiCad schematic)
At the start: 20 parts, among them SW1 SW_Push, U1 ATmega32U4-A, Y1 16MHz

Commit message: Save Progress
Parts:
- removed F1: 500mA, Fuse:Fuse_1206_3216Metric, symbol Device:Polyfuse
- removed USB1: Molex-0548190589, Connector_USB:USB_Micro-B_Molex-105133-0031, symbol random-keyboard-parts:Molex-0548190589
- added D1, D2: WS2812B, LED_SMD:LED_WS2812B-2020_PLCC4_2.0x2.0mm, symbol LED:WS2812B
- added F1: 500mA, Fuse:Fuse_1206_3216Metric, symbol Device:Polyfuse_Small
- added R7, R8: 5.1k, Resistor_SMD:R_0805_2012Metric, symbol Device:R_Small
- added U2: PRTR5V0U2X, Package_TO_SOT_SMD:SOT-143, symbol ai03-locallib:PRTR5V0U2X
- added USB1: HRO-TYPE-C-31-M-12, Type-C:HRO-TYPE-C-31-M-12-Assembly, symbol Voyager4-rescue:HRO-TYPE-C-31-M-12-Type-C
Connections:
- net +5V: now also D1.1 (VDD), D2.1 (VDD), F1.1
- net D+: now also U2.2 (IO1), USB1.6 (DP1), USB1.8 (DP2)
- net D-: now also U2.3 (IO2), USB1.5 (DN2), USB1.7 (DN1)
- net GND: now also D1.3 (VSS), D2.3 (VSS), R7.2, R8.2, U2.1 (GND), USB1.1 (GND), USB1.12 (GND), USB1.13 (SHIELD)
- net VCC: now also F1.2, U2.4 (VCC), USB1.11 (VBUS), USB1.2 (VBUS)
- net at U1.25 (PD4): now also MX1.2 (ROW), R5.2
- net RGBLED: now reaches U1.26 (PD6)
- net RGBLED: now also D1.4 (DIN)
- net at U1.32 (PC7): now also MX2.2 (ROW), R6.2
- new net: D1.2 (DOUT), D2.4 (DIN)
- new net: R7.1, USB1.10 (CC2)
- new net: R8.1, USB1.4 (CC1)
- now unconnected: U1.8 (PB0), U1.9 (PB1)
- no-connect marks 0 -> 24
