File: 2Key/2Key.kicad_sch (KiCad schematic)
At the start: 27 parts, among them SW1 SW_Push, U1 ATmega32U4-A, U2 PRTR5V0U2X, Y1 16MHz

Commit message: Updated PCB
Other:
- moved on the sheet: C8, C9
Changed lines of the file:
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@@
   (junction (at 194.945 127) (diameter 0) (color 0 0 0 0)
   )
+  (junction (at 142.24 86.36) (diameter 0) (color 0 0 0 0)
+  )
   (junction (at 196.215 124.46) (diameter 0) (color 0 0 0 0)
   )
@@
   (junction (at 200.025 158.115) (diameter 0) (color 0 0 0 0)
   )
-  (junction (at 144.78 86.36) (diameter 0) (color 0 0 0 0)
-  )
   (junction (at 93.98 34.29) (diameter 0) (color 0 0 0 0)
   )
@@
   (junction (at 66.04 54.61) (diameter 0) (color 0 0 0 0)
   )
-  (junction (at 144.78 81.28) (diameter 0) (color 0 0 0 0)
-  )
   (junction (at 163.83 86.36) (diameter 0) (color 0 0 0 0)
   )
@@
   )
   (junction (at 152.4 86.36) (diameter 0) (color 0 0 0 0)
+  )
+  (junction (at 142.24 81.28) (diameter 0) (color 0 0 0 0)
   )
   (junction (at 175.26 81.28) (diameter 0) (color 0 0 0 0)
@@
     (stroke (width 0) (type default) (color 0 0 0 0))
   )
-  (wire (pts (xy 144.78 86.36) (xy 152.4 86.36))
-    (stroke (width 0) (type default) (color 0 0 0 0))
-  )
   (wire (pts (xy 93.98 81.28) (xy 83.82 81.28))
     (stroke (width 0) (type default) (color 0 0 0 0))
   )
+  (wire (pts (xy 142.24 81.28) (xy 152.4 81.28))
+    (stroke (width 0) (type default) (color 0 0 0 0))
+  )
   (wire (pts (xy 73.66 73.66) (xy 83.82 73.66))
     (stroke (width 0) (type default) (color 0 0 0 0))
@@
     (stroke (width 0) (type default) (color 0 0 0 0))
   )
-  (wire (pts (xy 138.43 86.36) (xy 144.78 86.36))
+  (wire (pts (xy 132.08 86.36) (xy 142.24 86.36))
     (stroke (width 0) (type default) (color 0 0 0 0))
   )
@@
     (stroke (width 0) (type default) (color 0 0 0 0))
   )
+  (wire (pts (xy 142.24 86.36) (xy 152.4 86.36))
+    (stroke (width 0) (type default) (color 0 0 0 0))
+  )
   (wire (pts (xy 93.98 34.29) (xy 86.36 34.29))
     (stroke (width 0) (type default) (color 0 0 0 0))
@@
     (stroke (width 0) (type default) (color 0 0 0 0))
   )
-  (wire (pts (xy 144.78 81.28) (xy 152.4 81.28))
-    (stroke (width 0) (type default) (color 0 0 0 0))
-  )
   (wire (pts (xy 76.2 34.29) (xy 66.04 34.29))
     (stroke (width 0) (type default) (color 0 0 0 0))
@@
     (stroke (width 0) (type default) (color 0 0 0 0))
   )
-  (wire (pts (xy 138.43 81.28) (xy 144.78 81.28))
+  (wire (pts (xy 132.08 81.28) (xy 142.24 81.28))
     (stroke (width 0) (type default) (color 0 0 0 0))
   )
@@
     (pin "2")
   )
-  (symbol (lib_id "Device:C_Small") (at 144.78 83.82 0) (unit 1)
-    (in_bom yes) (on_board yes) (fields_autoplaced)
-    (property "Reference" "C9" (id 0) (at 147.32 82.5562 0)
-      (effects (font (size 1.27 1.27)) (justify left))
-    )
-    (property "Value" "0.1uF" (id 1) (at 147.32 85.0962 0)
-      (effects (font (size 1.27 1.27)) (justify left))
-    )
-    (property "Footprint" "Capacitor_SMD:C_0805_2012Metric" (id 2) (at 144.78 83.82 0)
-      (effects (font (size 1.27 1.27)) hide)
-    )
-    (property "Datasheet" "~" (id 3) (at 144.78 83.82 0)
+  (symbol (lib_id "Device:C_Small") (at 142.24 83.82 0) (unit 1)
+    (in_bom yes) (on_board yes) (fields_autoplaced)
+    (property "Reference" "C9" (id 0) (at 144.78 82.5562 0)
+      (effects (font (size 1.27 1.27)) (justify left))
+    )
+    (property "Value" "0.1uF" (id 1) (at 144.78 85.0962 0)
+      (effects (font (size 1.27 1.27)) (justify left))
+    )
+    (property "Footprint" "Capacitor_SMD:C_0805_2012Metric" (id 2) (at 142.24 83.82 0)
+      (effects (font (size 1.27 1.27)) hide)
+    )
+    (property "Datasheet" "~" (id 3) (at 142.24 83.82 0)
       (effects (font (size 1.27 1.27)) hide)
     )
@@
     (pin "2")
   )
-  (symbol (lib_id "Device:C_Small") (at 138.43 83.82 0) (unit 1)
-    (in_bom yes) (on_board yes) (fields_autoplaced)
-    (property "Reference" "C8" (id 0) (at 140.97 82.5562 0)
-      (effects (font (size 1.27 1.27)) (justify left))
-    )
-    (property "Value" "0.1uF" (id 1) (at 140.97 85.0962 0)
-      (effects (font (size 1.27 1.27)) (justify left))
-    )
-    (property "Footprint" "Capacitor_SMD:C_0805_2012Metric" (id 2) (at 138.43 83.82 0)
-      (effects (font (size 1.27 1.27)) hide)
-    )
-    (property "Datasheet" "~" (id 3) (at 138.43 83.82 0)
+  (symbol (lib_id "Device:C_Small") (at 132.08 83.82 0) (unit 1)
+    (in_bom yes) (on_board yes) (fields_autoplaced)
+    (property "Reference" "C8" (id 0) (at 134.62 82.5562 0)
+      (effects (font (size 1.27 1.27)) (justify left))
+    )
+    (property "Value" "0.1uF" (id 1) (at 134.62 85.0962 0)
+      (effects (font (size 1.27 1.27)) (justify left))
+    )
+    (property "Footprint" "Capacitor_SMD:C_0805_2012Metric" (id 2) (at 132.08 83.82 0)
+      (effects (font (size 1.27 1.27)) hide)
+    )
+    (property "Datasheet" "~" (id 3) (at 132.08 83.82 0)
       (effects (font (size 1.27 1.27)) hide)
     )
@@
   )
   (symbol (lib_id "power:+5V") (at 170.18 72.39 0) (unit 1)
-    (in_bom yes) (on_board yes) (fields_autoplaced)
+    (in_bom yes) (on_board yes)
     (property "Reference" "#PWR0117" (id 0) (at 170.18 76.2 0)
       (effects (font (size 1.27 1.27)) hide)
     )
-    (property "Value" "+5V" (id 1) (at 170.18 67.31 0))
+    (property "Value" "+5V" (id 1) (at 170.18 68.58 0))
     (property "Footprint" "" (id 2) (at 170.18 72.39 0)
       (effects (font (size 1.27 1.27)) hide)

Commit message: Remade PCB with the MU Chip
Remade the PCB with the MU Chip and switched to reverse mounted LEDs
Parts:
- removed D1, D2: WS2812B, LED_SMD:LED_WS2812B-2020_PLCC4_2.0x2.0mm, symbol LED:WS2812B
- removed U1: ATmega32U4-A, Package_QFP:TQFP-44_10x10mm_P0.8mm, symbol MCU_Microchip_ATmega:ATmega32U4-A
- added D1, D2: SK6812MINI, LED:SK6812MINIE, symbol LED:SK6812MINI
- added U1: ATmega32U4-M, Package_DFN_QFN:QFN-44-1EP_7x7mm_P0.5mm_EP5.2x5.2mm, symbol MCU_Microchip_ATmega:ATmega32U4-M
- C3: value C_Small -> 1uF
Connections:
- net +5V: now also D1.4 (VDD), D2.4 (VDD), U1.7 (VBUS)
- net GND: now also D1.2 (VSS), D2.2 (VSS), U1.15 (GND), U1.23 (GND), U1.35 (GND), U1.43 (GND), U1.45 (GND), U1.5 (UGND)
- net RGBLED: now also D1.3 (DIN), U1.26 (PD6)
- net VCC: now also U1.14 (VCC), U1.2 (UVCC), U1.24 (AVCC), U1.34 (VCC), U1.44 (AVCC)
- net at C2.2, Y1.1: now also U1.16 (XTAL2)
- net at C1.2, Y1.3: now also U1.17 (XTAL1)
- net at C3.1: now also U1.6 (UCAP)
- net at R3.2: now also U1.3 (D-)
- net at R4.2, SW1.2: now also U1.13 (~{RESET})
- net at MX1.2 (ROW), R5.2: now also U1.1 (PE6)
- net at MX2.2 (ROW), R6.2: now also U1.11 (PB3)
- net at R1.1: now also U1.33 (~{HWB}/PE2)
- net at R2.2: now also U1.4 (D+)
- new net: D1.1 (DOUT), D2.3 (DIN)
